Commit message: TO DO 3.4 of exercise
Correction bug on urdf file, write a listner to obtain: traslation, rotation matrix and axis angole rappresentation, and Eulero RYP.

Co-Authored-By: fabriziolettieri1 <58087395+fabriziolettieri1@users.noreply.github.com>
Co-Authored-By: veronicasalvati <73425251+veronicasalvati@users.noreply.github.com>
Co-Authored-By: ludus94 <l.russo62@studenti.unisa.it>

File: src/esercizio3_pkg/robot/fanuc.xacro (robot description, xacro)
@@ -139,5 +139,5 @@
         <!--Link properties-->
         <visual>
-            <origin xyz="-1.46 0 0.93" rpy="1.57 1.57 1.57" />
+            <origin xyz="1.46 0.001 -1.07" rpy="0 -1.57 0" />
             <geometry>
                 <mesh filename="package://esercizio3_pkg/meshes/visual/link_5.dae" />
@@ -146,5 +146,5 @@
         </visual>
         <collision>
-            <origin xyz="-1.46 0 0.93" rpy="1.57 1.57 1.57" />
+            <origin xyz="1.46 0.001 -1.07" rpy="0 -1.57 0" />
             <geometry>
                 <mesh filename="package://esercizio3_pkg/meshes/collision/link_5.stl" />
@@ -154,5 +154,5 @@
     <joint name="joint5" type="revolute">
         <!--Joint properties-->
-        <origin xyz="0 0.64 0.1" rpy="1.57 0 0" />
+        <origin xyz="0 0.64 0.1" rpy="1.57 1.57 0" />
         <parent link="link4" />
         <child link="link5" />
@@ -162,8 +162,8 @@
     </joint>
  <!--************************************************LINK 6********************************************-->
-    <link name="link6">
+    <link name="flange">
         <!--Link properties-->
         <visual>
-            <origin xyz="0 0 0" rpy="0 0 0" />
+            <origin xyz=" 0 0 -0.01" rpy="0 0 0" />
             <geometry>
                 <mesh filename="package://esercizio3_pkg/meshes/visual/link_6.dae" />
@@ -172,5 +172,5 @@
         </visual>
         <collision>
-            <origin xyz="0 0 0" rpy="0 0 0" />
+            <origin xyz="0 0 -0.01" rpy="0 0 0" />
             <geometry>
                 <mesh filename="package://esercizio3_pkg/meshes/collision/link_6.stl" />
@@ -178,9 +178,9 @@
         </collision>
     </link>
-    <joint name="joint6" type="revolute">
+    <joint name="joint6" type="fixed">
         <!--Joint properties-->
-        <origin xyz="0 0 -0.15" rpy="0 0 0" />
+        <origin xyz="0 0 -0.099" rpy="0 0 0" />
         <parent link="link5" />
-        <child link="link6" />
+        <child link="flange" />
         <axis xyz="0 0 1" />
         <limit lower="-6.28" upper="6.28" effort="5.8" velocity="11.0" />
@@ -188,10 +188,10 @@
     </joint>
 <!--************************************************FLANGE********************************************-->
-    <link name="flange"/>
+  <!--  <link name="flange"/>
     <joint name="flange" type="fixed">
-        <!--Joint properties-->
-        <origin xyz="0 0 0" rpy="0 0 0" />
+        Joint properties-->
+        <!--<origin xyz="0 0 -0.09" rpy="0 0 0" />
         <parent link="link6" />
         <child link="flange" />
-    </joint>
+    </joint>-->
 </robot>
